Commit message: 优化了dashboard的表现，并修复桥接节点文件的ROS信息bug

File: src/HRA_AFD_assmebly/urdf/HRA_AFD_assmebly.urdf (robot description, URDF)
Before this commit: robot HRA_AFD_assmebly, 16 links, 15 joints
Joints:
- joint AY+_joint: type continuous -> fixed
- joint AY-_joint: type continuous -> fixed
- joint FY+_joint: type continuous -> fixed
- joint FY-_joint: type continuous -> fixed
- joint LX+_joint: type continuous -> fixed
- joint LX-_joint: type continuous -> fixed
- joint LZ+_joint: type continuous -> fixed
- joint LZ-_joint: type continuous -> fixed
- joint RX+_joint: type continuous -> fixed
- joint RX-_joint: type continuous -> fixed
- joint RZ+_joint: type continuous -> fixed
- joint RZ-_joint: type continuous -> fixed

File: src/HRA_description/urdf/HRA_description.urdf (robot description, URDF)
Before this commit: robot HRA_description, 16 links, 15 joints
Joints:
- joint AY+_joint: type continuous -> fixed
- joint AY-_joint: type continuous -> fixed
- joint FY+_joint: type continuous -> fixed
- joint FY-_joint: type continuous -> fixed
- joint LX+_joint: type continuous -> fixed
- joint LX-_joint: type continuous -> fixed
- joint LZ+_joint: type continuous -> fixed
- joint LZ-_joint: type continuous -> fixed
- joint RX+_joint: type continuous -> fixed
- joint RX-_joint: type continuous -> fixed
- joint RZ+_joint: type continuous -> fixed
- joint RZ-_joint: type continuous -> fixed

Commit message: 修复了机器人-气足装配体的模型错误问题，并优化其URDF文件。

File: src/HRA_AFD_assmebly/urdf/HRA_AFD_assmebly.urdf (robot description, URDF)
Before this commit: robot HRA_AFD_assmebly, 16 links, 15 joints
Links:
- added link AFD_Link, mass 9.2544; collision mesh filename=package://HRA_AFD_assmebly/meshes/AFD_Link.STL; visual mesh filename=package://HRA_AFD_assmebly/meshes/AFD_Link.STL
- link dummy_link: mass 12.684 -> 3.4296
Joints:
- added joint AFD_joint: type fixed, parent base_link, child AFD_Link, origin xyz=0 0 -0.293 rpy=0 0 0, axis 0 0 1
- joint AY+_joint: origin xyz=-0.071 0.122 0.222 rpy=1.5708 0 -3.1416 -> xyz=-0.071 0.122 -0.071 rpy=1.5708 0 3.1416
- joint AY-_joint: origin xyz=-0.071 -0.122 0.364 rpy=1.5708 0 0 -> xyz=-0.071 -0.122 0.071 rpy=1.5708 0 0
- joint D435i_joint: origin xyz=0.11555 0.0175 0.3445 rpy=0 0 0 -> xyz=0.11555 0.0175 0.0515 rpy=0 0 0
- joint FY+_joint: origin xyz=0.071 0.122 0.364 rpy=1.5708 0 3.1416 -> xyz=0.071 0.122 0.071 rpy=1.5708 0 3.1416
- joint FY-_joint: origin xyz=0.071 -0.122 0.222 rpy=1.5708 0 0 -> xyz=0.071 -0.122 -0.071 rpy=1.5708 0 0
- joint LX+_joint: origin xyz=0.122 0.071 0.364 rpy=1.5708 0 1.5708 -> xyz=0.122 0.071 0.071 rpy=1.5708 0 1.5708
- joint LX-_joint: origin xyz=-0.122 0.071 0.222 rpy=1.5708 0 -1.5708 -> xyz=-0.122 0.071 -0.071 rpy=1.5708 0 -1.5708
- joint LZ+_joint: origin xyz=0.071 0.071 0.415 rpy=0 0 1.5708 -> xyz=0.071 0.071 0.122 rpy=0 0 1.5708
- joint LZ-_joint: origin xyz=-0.071 0.071 0.171 rpy=3.1416 0 -1.5708 -> xyz=-0.071 0.071 -0.122 rpy=3.1416 0 -1.5708
- joint RX+_joint: origin xyz=0.122 -0.071 0.222 rpy=1.5708 0 1.5708 -> xyz=0.122 -0.071 -0.071 rpy=1.5708 0 1.5708
- joint RX-_joint: origin xyz=-0.122 -0.071 0.364 rpy=1.5708 0 -1.5708 -> xyz=-0.122 -0.071 0.071 rpy=1.5708 0 -1.5708
- joint RZ+_joint: origin xyz=-0.071 -0.071 0.415 rpy=0 0 1.5708 -> xyz=-0.071 -0.071 0.122 rpy=0 0 1.5708
- joint RZ-_joint: origin xyz=0.071 -0.071 0.171 rpy=-3.1416 0 -1.5708 -> xyz=0.071 -0.071 -0.122 rpy=-3.1416 0 -1.5708
- joint T265_joint: origin xyz=0.1193 0 0.36925 rpy=0 0 0 -> xyz=0.1193 0 0.07625 rpy=0 0 0
